File: PCB/3Kxr's HackPad v1.1.kicad_pcb (KiCad board)
At the start: 2 copper layers, 78 x 58.3 mm, 9 parts, among them SW1 SW_Push, SW2 SW_Push, SW3 SW_Push, SW4 SW_Push, SW8 RotaryEncoder_Switch, U1 XIAO-RP2040-DIP

Commit message: update HackPad v1.1
Connections:
- net SDA renamed Net-(D1-DIN)
- SW8 pad A: Net-(U1-GPIO1/RX) -> Net-(U1-GPIO26/ADC0/A0)
- SW8 pad B: Net-(U1-GPIO2/SCK) -> Net-(U1-GPIO27/ADC1/A1)
- SW8 pad S1: Net-(U1-GPIO4/MISO) -> GND
- SW8 pad S2: Net-(U1-GPIO3/MOSI) -> Net-(U1-GPIO28/ADC2/A2)
- U1 pad 1: unconnected-(U1-GPIO26/ADC0/A0-Pad1) -> Net-(U1-GPIO26/ADC0/A0)
- U1 pad 2: unconnected-(U1-GPIO27/ADC1/A1-Pad2) -> Net-(U1-GPIO27/ADC1/A1)
- U1 pad 3: unconnected-(U1-GPIO28/ADC2/A2-Pad3) -> Net-(U1-GPIO28/ADC2/A2)
- U1 pad 6: SCL -> unconnected-(U1-GPIO7/SCL-Pad6)
Routing:
- net Net-(U1-GPIO28/ADC2/A2): track 0.00 -> 80.9 mm, vias 0 -> 1
- net Net-(U1-GPIO26/ADC0/A0): track 0.00 -> 78.4 mm
- net Net-(U1-GPIO27/ADC1/A1): track 0.00 -> 68.6 mm, vias 0 -> 1
- net Net-(U1-GPIO2/SCK): track 78.2 -> 33.1 mm, vias 3 -> 0
- net Net-(U1-GPIO4/MISO): track 85.4 -> 52.6 mm, vias 2 -> 1
- net GND: track 114.8 -> 146.7 mm, vias 5 -> 4
- net Net-(U1-GPIO3/MOSI): track 104.4 -> 80.6 mm
- net Net-(U1-GPIO1/RX): track 48.1 -> 36.3 mm, vias 1 -> 3
- net Net-(D1-DOUT): track 20.2 -> 22.6 mm, vias 3 -> 2
- net Net-(D1-DIN): track 32.3 -> 34.2 mm, vias 0 -> 2
- net +5V: track 36.9 -> 36.2 mm

Commit message: refactor: replace SK6812MINI with SK6812MINI-E and reorganize the circuit
Parts:
- removed D1, D2: SK6812MINI, LED_SMD:LED_SK6812MINI_PLCC4_3.5x3.5mm_P1.75mm
- added D3: SK6812MINI-E, SK6812MINI-E:SK6812MINI-E_fixed, F.Cu at (149.5, 64.1)
- added D4: SK6812MINI-E, SK6812MINI-E:SK6812MINI-E_fixed, F.Cu at (149.4, 71.5)
Routing:
- net Net-(U1-GPIO27/ADC1/A1): track 68.6 -> 120.0 mm
- net Net-(U1-GPIO4/MISO): track 52.6 -> 80.0 mm
- net Net-(D1-DOUT): track 22.6 -> 0.00 mm, vias 2 -> 0
- net Net-(D3-DIN): track 34.2 -> 56.3 mm, vias 2 -> 1
- net Net-(U1-GPIO3/MOSI): track 80.6 -> 59.9 mm, vias 0 -> 2
- net Net-(U1-GPIO26/ADC0/A0): track 78.4 -> 68.0 mm, vias 0 -> 3
- net GND: track 146.7 -> 139.2 mm, vias 4 -> 3
- net Net-(U1-GPIO1/RX): track 36.3 -> 30.3 mm, vias 3 -> 2
- net Net-(U1-GPIO28/ADC2/A2): track 80.9 -> 86.8 mm, vias 1 -> 2
- net +5V: track 36.2 -> 41.0 mm
- net Net-(U1-GPIO2/SCK): track 33.1 -> 33.6 mm

Commit message: fix: resolve unconnected circuit issue
Routing:
- net Net-(D3-DOUT): track 0.00 -> 11.3 mm
- net +5V: track 41.0 -> 40.2 mm
Changed lines of the file:
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@@
-	)
-	(segment
-		(start 146.87 63.23)
-		(end 146.31 62.67)
-		(width 0.2)
-		(layer "B.Cu")
-		(net 1)
 	)
 	(segment
@@
 	)
 	(segment
+		(start 146.87 67.3)
+		(end 146.87 64.73)
+		(width 0.2)
+		(layer "B.Cu")
+		(net 14)
+	)
+	(segment
+		(start 146.77 67.4)
+		(end 146.87 67.3)
+		(width 0.2)
+		(layer "B.Cu")
+		(net 14)
+	)
+	(segment
+		(start 152 70.62)
+		(end 152.19 70.43)
+		(width 0.2)
+		(layer "B.Cu")
+		(net 14)
+	)
+	(segment
+		(start 152.19 70.43)
+		(end 152.19 67.59)
+		(width 0.2)
+		(layer "B.Cu")
+		(net 14)
+	)
+	(segment
+		(start 152.19 67.59)
+		(end 146.96 67.59)
+		(width 0.2)
+		(layer "B.Cu")
+		(net 14)
+	)
+	(segment
+		(start 146.96 67.59)
+		(end 146.77 67.4)
+		(width 0.2)
+		(layer "B.Cu")
+		(net 14)
+	)
+	(segment

Commit message: reorganize the circuit
Routing:
- net +5V: track 40.2 -> 41.0 mm
